File: kicad/LoRa_prototype/antenna.kicad_sch (KiCad schematic)
At the start: 5 parts, among them J2 U.FL, U3 AS179-92LF

Commit message: Copied and cleaned up USb charging circuit from WORK-CARE
1 ERC error
Parts:
- renumbered C22 to C35, C23 to C36, C27 to C37, J2 to J4, U3 to U5
Changed lines of the file:
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@@
 		(on_board yes)
 		(dnp no)
-		(property "Reference" "#PWR019"
+		(property "Reference" "#PWR055"
 			(at 148.59 104.14 0)
 			(effects
@@
 			(project "LoRa_prototype"
 				(path "/9fad4700-f514-47ad-821a-b4076ecc08de/724a66f0-96b6-4d19-9e27-2d301e795177"
-					(reference "#PWR019")
+					(reference "#PWR055")
 					(unit 1)
 				)
@@
 		(on_board yes)
 		(dnp no)
-		(property "Reference" "#PWR018"
+		(property "Reference" "#PWR054"
 			(at 124.46 81.28 0)
 			(effects
@@
 			(project "LoRa_prototype"
 				(path "/9fad4700-f514-47ad-821a-b4076ecc08de/724a66f0-96b6-4d19-9e27-2d301e795177"
-					(reference "#PWR018")
+					(reference "#PWR054")
 					(unit 1)
 				)
@@
 		(on_board yes)
 		(dnp no)
-		(property "Reference" "U3"
+		(property "Reference" "U5"
 			(at 122.936 95.25 0)
 			(effects
@@
 			(project "LoRa_prototype"
 				(path "/9fad4700-f514-47ad-821a-b4076ecc08de/724a66f0-96b6-4d19-9e27-2d301e795177"
-					(reference "U3")
+					(reference "U5")
 					(unit 1)
 				)
@@
 		(dnp no)
 		(fields_autoplaced yes)
-		(property "Reference" "J2"
+		(property "Reference" "J4"
 			(at 151.13 89.1931 0)
 			(effects
@@
 			(project "LoRa_prototype"
 				(path "/9fad4700-f514-47ad-821a-b4076ecc08de/724a66f0-96b6-4d19-9e27-2d301e795177"
-					(reference "J2")
+					(reference "J4")
 					(unit 1)
 				)
@@
 		(on_board yes)
 		(dnp no)
-		(property "Reference" "C23"
+		(property "Reference" "C36"
 			(at 107.95 96.52 90)
 			(effects
@@
 			(project "LoRa_prototype"
 				(path "/9fad4700-f514-47ad-821a-b4076ecc08de/724a66f0-96b6-4d19-9e27-2d301e795177"
-					(reference "C23")
+					(reference "C36")
 					(unit 1)
 				)
@@
 		(on_board yes)
 		(dnp no)
-		(property "Reference" "C27"
+		(property "Reference" "C37"
 			(at 137.16 93.98 90)
 			(effects
@@
 			(project "LoRa_prototype"
 				(path "/9fad4700-f514-47ad-821a-b4076ecc08de/724a66f0-96b6-4d19-9e27-2d301e795177"
-					(reference "C27")
+					(reference "C37")
 					(unit 1)
 				)
@@
 		(on_board yes)
 		(dnp no)
-		(property "Reference" "C22"
+		(property "Reference" "C35"
 			(at 107.95 82.042 90)
 			(effects
@@
 			(project "LoRa_prototype"
 				(path "/9fad4700-f514-47ad-821a-b4076ecc08de/724a66f0-96b6-4d19-9e27-2d301e795177"
-					(reference "C22")
-					(unit 1)
-				)
+					(reference "C35")
+					(unit 1)
+				)
