File: kicad/LoRa_prototype/antenna.kicad_sch (KiCad schematic)
At the start: 5 parts, among them J4 U.FL, U5 AS179-92LF

Commit message: Created separate folders for footprints and 3d models
Parts:
- C35, C36, C37: footprint (none) -> Capacitor_SMD:C_0805_2012Metric
Changed lines of the file:
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@@
 			)
 		)
-		(property "Footprint" ""
+		(property "Footprint" "Capacitor_SMD:C_0805_2012Metric"
 			(at 111.76 91.7448 0)
 			(effects
@@
 			)
 		)
-		(property "Footprint" ""
+		(property "Footprint" "Capacitor_SMD:C_0805_2012Metric"
 			(at 140.97 89.2048 0)
 			(effects
@@
 			)
 		)
-		(property "Footprint" ""
+		(property "Footprint" "Capacitor_SMD:C_0805_2012Metric"
 			(at 111.76 86.6648 0)
 			(effects

Commit message: Assigned almost all footprints
Parts:
- J4: footprint PCM_JLCPCB:IPEX-SMD_BWIPX-1-001E -> (none)
Changed lines of the file:
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@@
 			)
 		)
-		(property "Footprint" "PCM_JLCPCB:IPEX-SMD_BWIPX-1-001E"
+		(property "Footprint" ""
 			(at 148.59 90.17 0)
 			(hide yes)

Commit message: Assigned all footprints
Parts:
- added C10, C7: C, Capacitor_SMD:C_0201_0603Metric, symbol Device:C
- added L8: 0, Inductor_SMD:L_0603_1608Metric, symbol Device:L
- added R2: 0, Resistor_SMD:R_0603_1608Metric, symbol Device:R
- J4: value U.FL -> SMA Female; footprint (none) -> Connector_Coaxial:SMA_Samtec_SMA-J-P-H-ST-EM1_EdgeMount
Connections:
- net GND: now also C10.2, C7.2
- net at J4.1 (In): now also C10.1, L8.2; no longer C37.2
- new net: C7.1, L8.1, R2.2
- new net: C37.2, R2.1
Other:
- note added: "Pi-network for manual tuning"
- moved on the sheet: J4
